Commit message: Fixed failures in simulated robot and added pkg for real robot

File: ur5e_cam-grippers_simulated_moveit_config/config/gazebo_ur5e_cam.urdf (robot description, URDF)
Before this commit: robot ur5e_cam, 31 links, 30 joints
Joints:
- joint gripper_joint: origin xyz=0.01 0.0125 0 rpy=0 1.5708 0 -> xyz=0 0 0 rpy=0 0 0
- joint gripper_joint1: origin xyz=0.01 -0.0125 0 rpy=0 1.5708 0 -> xyz=0 0.0125 0 rpy=0 0 0
- joint gripper_joint2: origin xyz=0.01 0 0.0125 rpy=0 1.5708 0 -> xyz=0 -0.0125 0 rpy=0 0 0
- joint gripper_joint3: origin xyz=0.01 0 -0.0125 rpy=0 1.5708 0 -> xyz=0.0125 0 0 rpy=0 0 0
- joint gripper_joint4: origin xyz=0.01 0 0 rpy=0 1.5708 0 -> xyz=-0.0125 0 0 rpy=0 0 0
- joint gripper_joint5: origin xyz=0.01 0.0125 0.0125 rpy=0 1.5708 0 -> xyz=0.0125 0.0125 0 rpy=0 0 0
- joint gripper_joint6: origin xyz=0.01 -0.0125 0.0125 rpy=0 1.5708 0 -> xyz=-0.0125 0.0125 0 rpy=0 0 0
- joint gripper_joint7: origin xyz=0.01 0.0125 -0.0125 rpy=0 1.5708 0 -> xyz=0.0125 -0.0125 0 rpy=0 0 0
- joint gripper_joint8: origin xyz=0.01 -0.0125 -0.0125 rpy=0 1.5708 0 -> xyz=-0.0125 -0.0125 0 rpy=0 0 0

File: ur5e_cam_description/urdf/grippers.urdf.xacro (robot description, xacro)
@@ -23,5 +23,5 @@
             <parent link="${parent}" />
             <child link="vacuum_gripper" />
-            <origin rpy="0 1.5708 0" xyz="0.01 0.0125 0" />
+            <origin rpy="0 0 0" xyz="0 0 0" />
             <limit effort="50" velocity="50" lower="0" upper="0" />
             <dynamics damping="0.0" friction="10"/>
@@ -58,5 +58,5 @@
         <parent link="${parent}" />
         <child link="vacuum_gripper1" />
-        <origin rpy="0 1.5708 0" xyz="0.01 -0.0125 0" />
+        <origin rpy="0 0 0" xyz="0 0.0125 0" />
         <limit effort="50" velocity="50" lower="0" upper="0" />
         <dynamics damping="0.0" friction="10"/>
@@ -93,5 +93,5 @@
         <parent link="${parent}" />
         <child link="vacuum_gripper2" />
-        <origin rpy="0 1.5708 0" xyz="0.01 0 0.0125" />
+        <origin rpy="0 0 0" xyz="0 -0.0125 0" />
         <limit effort="50" velocity="50" lower="0" upper="0" />
         <dynamics damping="0.0" friction="10"/>
@@ -128,5 +128,5 @@
         <parent link="${parent}" />
         <child link="vacuum_gripper3" />
-        <origin rpy="0 1.5708 0" xyz="0.01 0 -0.0125" />
+        <origin rpy="0 0 0" xyz="0.0125 0 0" />
         <limit effort="50" velocity="50" lower="0" upper="0" />
         <dynamics damping="0.0" friction="10"/>
@@ -163,5 +163,5 @@
             <parent link="${parent}" />
             <child link="vacuum_gripper4" />
-            <origin rpy="0 1.5708 0" xyz="0.01 0 0" />
+            <origin rpy="0 0 0" xyz="-0.0125 0 0" />
             <limit effort="50" velocity="50" lower="0" upper="0" />
             <dynamics damping="0.0" friction="10"/>
@@ -198,5 +198,5 @@
             <parent link="${parent}" />
             <child link="vacuum_gripper5" />
-            <origin rpy="0 1.5708 0" xyz="0.01 0.0125 0.0125" />
+            <origin rpy="0 0 0" xyz="0.0125 0.0125 0" />
             <limit effort="50" velocity="50" lower="0" upper="0" />
             <dynamics damping="0.0" friction="10"/>
@@ -233,5 +233,5 @@
             <parent link="${parent}" />
             <child link="vacuum_gripper6" />
-            <origin rpy="0 1.5708 0" xyz="0.01 -0.0125 0.0125" />
+            <origin rpy="0 0 0" xyz="-0.0125 0.0125 0" />
             <limit effort="50" velocity="50" lower="0" upper="0" />
             <dynamics damping="0.0" friction="10"/>
@@ -268,5 +268,5 @@
             <parent link="${parent}" />
             <child link="vacuum_gripper7" />
-            <origin rpy="0 1.5708 0" xyz="0.01 0.0125 -0.0125" />
+            <origin rpy="0 0 0" xyz="0.0125 -0.0125 0" />
             <limit effort="50" velocity="50" lower="0" upper="0" />
             <dynamics damping="0.0" friction="10"/>
@@ -303,5 +303,5 @@
             <parent link="${parent}" />
             <child link="vacuum_gripper8" />
-            <origin rpy="0 1.5708 0" xyz="0.01 -0.0125 -0.0125" />
+            <origin rpy="0 0 0" xyz="-0.0125 -0.0125 0" />
             <limit effort="50" velocity="50" lower="0" upper="0" />
             <dynamics damping="0.0" friction="10"/>

File: ur5e_cam_description/urdf/ur5e_robot_camera-grippers_sim.urdf.xacro (robot description, xacro)
@@ -53,5 +53,5 @@
   <!-- camera -->
   <xacro:arg name="use_nominal_extrinsics" default="false" />
-  <xacro:include filename="$(find realsense2_description)/urdf/_d435.urdf.xacro"/>
+  <xacro:include filename="$(find realsense2_description_issaias)/urdf/_d435.urdf.xacro"/>
   <xacro:sensor_d435 parent="wrist_3_link">
     <origin xyz="0.0 0.045 -0.03" rpy="0 0.0 1.57"/>

File: ur5e_cam_description/urdf/ur5e_robot_camera_sim.urdf.xacro (robot description, xacro)
@@ -53,5 +53,5 @@
   <!-- camera -->
   <xacro:arg name="use_nominal_extrinsics" default="false" />
-  <xacro:include filename="$(find realsense2_description)/urdf/_d435.urdf.xacro"/>
+  <xacro:include filename="$(find realsense2_description_issaias)/urdf/_d435.urdf.xacro"/>
   <xacro:sensor_d435 parent="wrist_3_link">
     <origin xyz="0.0 0.045 -0.03" rpy="0 0.0 1.57"/>
