Commit message: Vacuum grippers update

File: ur5e_cam_description/urdf/grippers.urdf.xacro (robot description, xacro)
@@ -1,29 +1,29 @@
 <?xml version="1.0"?>
-<robot xmlns:xacro="http://ros.org/wiki/xacro">
+<robot name="grippers" xmlns:xacro="http://ros.org/wiki/xacro">
     <xacro:macro name="grippers" params="parent">
         <link name="vacuum_gripper">
-        <gravity>0</gravity>
-        <visual>
-            <origin rpy="0 0 0" xyz="0 0 0"/>
-            <geometry>
-            <cylinder radius="0.005" length="0.01"/>
-            </geometry>
-            <material name="transparent">
-            <color rgba="0 0 0 0"/>
-            </material>
-        </visual>
-        <inertial>
-            <origin rpy="0 0 0" xyz="0.000000 0.000000 0.000000"/>
-            <mass value="0.0001"/>
-            <inertia ixx="1e-08" ixy="0" ixz="0" iyy="1e-08" iyz="0" izz="1e-08"/>
-        </inertial>
+            <gravity>0</gravity>
+            <visual>
+                <origin rpy="0 0 0" xyz="0 0 0"/>
+                <geometry>
+                    <cylinder radius="0.005" length="0.01"/>
+                </geometry>
+                <material name="transparent">
+                    <color rgba="0 0 0 0"/>
+                </material>
+            </visual>
+            <inertial>
+                <origin rpy="0 0 0" xyz="0.000000 0.000000 0.000000"/>
+                <mass value="0.0001"/>
+                <inertia ixx="1e-08" ixy="0" ixz="0" iyy="1e-08" iyz="0" izz="1e-08"/>
+            </inertial>
         </link>
         <joint name="gripper_joint" type="revolute">
-        <axis xyz="1 0 0" />
-        <parent link="${parent}" />
-        <child link="vacuum_gripper" />
-        <origin rpy="0 1.5708 0" xyz="0.01 0.0125 0" />
-        <limit effort="50" velocity="50" lower="0" upper="0" />
-        <dynamics damping="0.0" friction="10"/>
+            <axis xyz="1 0 0" />
+            <parent link="${parent}" />
+            <child link="vacuum_gripper" />
+            <origin rpy="0 1.5708 0" xyz="0.01 0.0125 0" />
+            <limit effort="50" velocity="50" lower="0" upper="0" />
+            <dynamics damping="0.0" friction="10"/>
         </joint>
         <gazebo>
@@ -37,5 +37,5 @@
             </plugin>
         </gazebo>
-        <link name="vacuum_gripper1">
+        <!-- <link name="vacuum_gripper1">
         <gravity>0</gravity>
         <visual>
@@ -316,5 +316,5 @@
             <minDistance>0.01</minDistance>
             </plugin>
-        </gazebo>
+        </gazebo> -->
     </xacro:macro>
 </robot>

File: ur5e_cam_description/urdf/ur5e_robot_camera-grippers_sim.urdf.xacro (robot description, xacro)
@@ -1,16 +1,53 @@
 <?xml version="1.0"?>
 <robot xmlns:xacro="http://ros.org/wiki/xacro"
-       name="ur5e" >
-  <!-- common stuff -->
-  <xacro:include filename="$(find ur_e_description)/urdf/common.gazebo.xacro" />
-  <!-- ur5e -->
-  <xacro:include filename="$(find ur_description)/urdf/inc/ur5_macro.xacro"/>
-  <!-- arm -->
-  <xacro:ur5_robot prefix="" />
-  <link name="world" />
+       name="ur5e_cam" >
+  <!-- LAUNCHING GAZEBO MODEL -->
+  <!--
+    Import main macro.
+    NOTE: this imports the Gazebo-wrapper main macro, NOT the regular
+          xacro macro (which is hosted by ur_description).
+  -->
+  <xacro:include filename="$(find ur_gazebo)/urdf/ur_macro.xacro"/>
+  <!--Declare arguments -->
+  <xacro:arg name="joint_limit_params" default="$(find ur_description)/config/ur5/joint_limits.yaml"/>
+  <xacro:arg name="physical_params" default="$(find ur_description)/config/ur5/physical_parameters.yaml"/>
+  <xacro:arg name="kinematics_params" default="$(find ur_description)/config/ur5/default_kinematics.yaml"/>
+  <xacro:arg name="visual_params" default="$(find ur_description)/config/ur5/visual_parameters.yaml"/>
+  <!--
+    legal values:
+      - hardware_interface/PositionJointInterface
+      - hardware_interface/VelocityJointInterface
+      - hardware_interface/EffortJointInterface
+    NOTE: this value must correspond to the controller configured in the
+          controller .yaml files in the 'config' directory.
+  -->
+  <xacro:arg name="transmission_hw_interface" default="hardware_interface/PositionJointInterface"/>
+  <xacro:arg name="safety_limits" default="false"/>
+  <xacro:arg name="safety_pos_margin" default="0.15"/>
+  <xacro:arg name="safety_k_position" default="20"/>
+  <!-- Instantiate the Gazebo robot and pass it all the required arguments. -->
+  <xacro:ur_robot_gazebo
+    prefix=""
+    joint_limits_parameters_file="$(arg joint_limit_params)"
+    kinematics_parameters_file="$(arg kinematics_params)"
+    physical_parameters_file="$(arg physical_params)"
+    visual_parameters_file="$(arg visual_params)"
+    transmission_hw_interface="$(arg transmission_hw_interface)"
+    safety_limits="$(arg safety_limits)"
+    safety_pos_margin="$(arg safety_pos_margin)"
+    safety_k_position="$(arg safety_k_position)"
+  />
+  <!--
+    Attach the Gazebo model to Gazebo's world frame.
+    Note: if you're looking to integrate a UR into a larger scene and need
+    to add EEFs or other parts, DO NOT change this file or the 'world' link
+    here. Create a NEW xacro instead and decide whether you need to add
+    a 'world' link there.
+  -->
+  <link name="world"/>
   <joint name="world_joint" type="fixed">
-    <parent link="world" />
-    <child link = "base_link" />
-    <origin xyz="0.0 0.0 0.0" rpy="0.0 0.0 0.0" />
+    <parent link="world"/>
+    <child link="base_link"/>
+    <origin xyz="0 0 0" rpy="0 0 0"/>
   </joint>
   <!-- camera -->
@@ -22,5 +59,5 @@
   <!-- vacuum gripper -->
   <xacro:include filename="$(find ur5e_cam_description)/urdf/grippers.urdf.xacro"/>
-  <xacro:grippers parent="tool0">
+  <xacro:grippers parent="wrist_3_link">
   </xacro:grippers>
 </robot>

Commit message: Fallo en pasar a tf la detección

File: ur5e_cam_description/urdf/grippers.urdf.xacro (robot description, xacro)
@@ -37,5 +37,5 @@
             </plugin>
         </gazebo>
-        <!-- <link name="vacuum_gripper1">
+        <link name="vacuum_gripper1">
         <gravity>0</gravity>
         <visual>
@@ -316,5 +316,5 @@
             <minDistance>0.01</minDistance>
             </plugin>
-        </gazebo> -->
+        </gazebo>
     </xacro:macro>
 </robot>

Commit message: Fixed IK errors and updated VA developments

File: ur5e_cam_description/urdf/grippers.urdf.xacro (robot description, xacro)
@@ -1,5 +1,5 @@
 <?xml version="1.0"?>
 <robot name="grippers" xmlns:xacro="http://ros.org/wiki/xacro">
-    <xacro:macro name="grippers" params="parent">
+    <xacro:macro name="grippers" params="parent z:=0">
         <link name="vacuum_gripper">
             <gravity>0</gravity>
@@ -23,5 +23,5 @@
             <parent link="${parent}" />
             <child link="vacuum_gripper" />
-            <origin rpy="0 0 0" xyz="0 0 0" />
+            <origin rpy="0 0 0" xyz="0 0 ${z}" />
             <limit effort="50" velocity="50" lower="0" upper="0" />
             <dynamics damping="0.0" friction="10"/>
@@ -58,5 +58,5 @@
         <parent link="${parent}" />
         <child link="vacuum_gripper1" />
-        <origin rpy="0 0 0" xyz="0 0.0125 0" />
+        <origin rpy="0 0 0" xyz="0 0.0125 ${z}" />
         <limit effort="50" velocity="50" lower="0" upper="0" />
         <dynamics damping="0.0" friction="10"/>
@@ -93,5 +93,5 @@
         <parent link="${parent}" />
         <child link="vacuum_gripper2" />
-        <origin rpy="0 0 0" xyz="0 -0.0125 0" />
+        <origin rpy="0 0 0" xyz="0 -0.0125 ${z}" />
         <limit effort="50" velocity="50" lower="0" upper="0" />
         <dynamics damping="0.0" friction="10"/>
@@ -128,5 +128,5 @@
         <parent link="${parent}" />
         <child link="vacuum_gripper3" />
-        <origin rpy="0 0 0" xyz="0.0125 0 0" />
+        <origin rpy="0 0 0" xyz="0.0125 0 ${z}" />
         <limit effort="50" velocity="50" lower="0" upper="0" />
         <dynamics damping="0.0" friction="10"/>
@@ -163,5 +163,5 @@
             <parent link="${parent}" />
             <child link="vacuum_gripper4" />
-            <origin rpy="0 0 0" xyz="-0.0125 0 0" />
+            <origin rpy="0 0 0" xyz="-0.0125 0 ${z}" />
             <limit effort="50" velocity="50" lower="0" upper="0" />
             <dynamics damping="0.0" friction="10"/>
@@ -198,5 +198,5 @@
             <parent link="${parent}" />
             <child link="vacuum_gripper5" />
-            <origin rpy="0 0 0" xyz="0.0125 0.0125 0" />
+            <origin rpy="0 0 0" xyz="0.0125 0.0125 ${z}" />
             <limit effort="50" velocity="50" lower="0" upper="0" />
             <dynamics damping="0.0" friction="10"/>
@@ -233,5 +233,5 @@
             <parent link="${parent}" />
             <child link="vacuum_gripper6" />
-            <origin rpy="0 0 0" xyz="-0.0125 0.0125 0" />
+            <origin rpy="0 0 0" xyz="-0.0125 0.0125 ${z}" />
             <limit effort="50" velocity="50" lower="0" upper="0" />
             <dynamics damping="0.0" friction="10"/>
@@ -268,5 +268,5 @@
             <parent link="${parent}" />
             <child link="vacuum_gripper7" />
-            <origin rpy="0 0 0" xyz="0.0125 -0.0125 0" />
+            <origin rpy="0 0 0" xyz="0.0125 -0.0125 ${z}" />
             <limit effort="50" velocity="50" lower="0" upper="0" />
             <dynamics damping="0.0" friction="10"/>
@@ -303,5 +303,5 @@
             <parent link="${parent}" />
             <child link="vacuum_gripper8" />
-            <origin rpy="0 0 0" xyz="-0.0125 -0.0125 0" />
+            <origin rpy="0 0 0" xyz="-0.0125 -0.0125 ${z}" />
             <limit effort="50" velocity="50" lower="0" upper="0" />
             <dynamics damping="0.0" friction="10"/>
